Commit message: del visual

File: src/urdf5/urdf/urdf5.urdf (robot description, URDF)
Before this commit: robot urdf5, 5 links, 4 joints
Links:
- link base_link: geometry collision mesh filename=package://urdf5/meshes/base_link.STL
- link imu_link: geometry collision mesh filename=package://urdf5/meshes/imu_link.STL
- link left_wheel_link: geometry collision mesh filename=package://urdf5/meshes/left_wheel_link.STL
- link lidar_link: geometry collision mesh filename=package://urdf5/meshes/lidar_link.STL
- link right_wheel_link: geometry collision mesh filename=package://urdf5/meshes/right_wheel_link.STL
