Commit message: urdfv6

File: src/robot_description_v6/urdf/robot_description_v6.urdf (robot description, URDF)
Before this commit: robot robot_description_v5, 6 links, 5 joints
Links:
- link base_link: mass 10.7166420111859 -> 9.39619068658646; geometry collision mesh filename=package://robot_description_v6/meshes/base_link.STL; visual mesh filename=package://robot_description_v6/meshes/base_link.STL
- link camera_link: geometry collision mesh filename=package://robot_description_v6/meshes/camera_link.STL; visual mesh filename=package://robot_description_v6/meshes/camera_link.STL
- link imu_link: mass 0.000999898118986841 -> 0.00712049275087492; geometry collision mesh filename=package://robot_description_v6/meshes/imu_link.STL; visual mesh filename=package://robot_description_v6/meshes/imu_link.STL
- link left_wheel_link: geometry collision mesh filename=package://robot_description_v6/meshes/left_wheel_link.STL; visual mesh filename=package://robot_description_v6/meshes/left_wheel_link.STL
- link lidar_link: mass 0.0312409127404856 -> 0.0312409127404862; geometry collision mesh filename=package://robot_description_v6/meshes/lidar_link.STL; visual mesh filename=package://robot_description_v6/meshes/lidar_link.STL
- link right_wheel_link: mass 0.981706650902444 -> 0.98170665090244; geometry collision mesh filename=package://robot_description_v6/meshes/right_wheel_link.STL; visual mesh filename=package://robot_description_v6/meshes/right_wheel_link.STL
Joints:
- joint imu: axis 0 0 0 -> 0 0 1; origin xyz=0.126428933055049 -0.100523077234269 0.0330200000034927 rpy=0 0 0 -> xyz=0.15399361324347 -0.0854574244366719 0.0409999999999995 rpy=0 0 0; type fixed -> continuous
- joint right_wheel: origin xyz=0.00157556970077088 -0.175020257687692 0.0150000000042174 rpy=0 0 0 -> xyz=0.00157556970077044 -0.175020257687692 0.0150000000042175 rpy=0 0 0
