Commit message: urdfv6

File: src/robot_description_v7/urdf/robot_description_v7.urdf (robot description, URDF)
Before this commit: robot robot_description_v6, 6 links, 5 joints
Links:
- link base_link: mass 9.39619068658646 -> 9.39619068658661; geometry collision mesh filename=package://robot_description_v7/meshes/base_link.STL; visual mesh filename=package://robot_description_v7/meshes/base_link.STL
- link camera_link: geometry collision mesh filename=package://robot_description_v7/meshes/camera_link.STL; visual mesh filename=package://robot_description_v7/meshes/camera_link.STL
- link imu_link: geometry collision mesh filename=package://robot_description_v7/meshes/imu_link.STL; visual mesh filename=package://robot_description_v7/meshes/imu_link.STL
- link left_wheel_link: geometry collision mesh filename=package://robot_description_v7/meshes/left_wheel_link.STL; visual mesh filename=package://robot_description_v7/meshes/left_wheel_link.STL
- link lidar_link: mass 0.0312409127404862 -> 0.0312409127406477; geometry collision mesh filename=package://robot_description_v7/meshes/lidar_link.STL; visual mesh filename=package://robot_description_v7/meshes/lidar_link.STL
- link right_wheel_link: geometry collision mesh filename=package://robot_description_v7/meshes/right_wheel_link.STL; visual mesh filename=package://robot_description_v7/meshes/right_wheel_link.STL
Joints:
- joint imu: axis 0 0 1 -> 0 0 0; origin xyz=0.15399361324347 -0.0854574244366719 0.0409999999999995 rpy=0 0 0 -> xyz=0.15399 -0.085457 0.041 rpy=0 0 0; type continuous -> fixed
- joint left_wheel: axis 0.00825691107326281 -0.999965911128739 0 -> 0.0082569 -0.99997 0; origin xyz=-0.00131434917487327 0.174967811207364 0.0150000000042175 rpy=0 0 0 -> xyz=-0.0013143 0.17497 0.015 rpy=0 0 0
- joint right_wheel: axis -0.00825691107326283 0.999965911128739 0 -> -0.0082569 0.99997 0; origin xyz=0.00157556970077044 -0.175020257687692 0.0150000000042175 rpy=0 0 0 -> xyz=0.0015756 -0.17502 0.015 rpy=0 0 0
